File: mini_project_3/iCE40UP5Kdev/iCE40UP5Kdev.kicad_pcb (KiCad board)
At the start: 2 copper layers, 25.4 x 52.1 mm, 52 parts, among them J1 USB4105-GF-A, J2 Left, J3 Right, U1 W25Q32JV, U2 MIC5365-1-2YD5, U3 MIC5318-3-3YD5, U4 ICE40UP5K-SG48ITR, X1 IQXO-791

Commit message: Add minor layout changes to MP3
Parts:
- moved R11 16.9 mm to (149.4, 92.2), turned to -90 degrees
- moved R4 0.51 mm to (152.0, 96.1)
- moved D2 0.51 mm to (150.1, 96.1)
- moved R3 0.23 mm to (151.3, 92.3)
- moved C13 0.05 mm to (155.7, 116.7)
Routing:
- net Net-(U4-IOB_23b): track 4.45 -> 32.5 mm, vias 0 -> 2
- net Net-(J1-D+-PadA6): track 55.5 -> 32.6 mm, vias 2 -> 0
- net +1V2: track 40.6 -> 39.3 mm, vias 8 -> 7
- net +3V3: track 181.3 -> 180.6 mm
- net +5V: track 50.8 -> 50.2 mm
Other:
- board size 25.4 x 52.1 mm -> 25.4 x 52.4 mm
